File: proyecto/car1/car1.kicad_sch (KiCad schematic)
At the start: 26 parts, among them J1 HC-sr04, J10 vcc Edu ciaa, J11 Adafruit A, J12 Adafruit B, J2 HC-sr04, J3 HC-sr04, J4 usb c socket, J5 SERVO, J6 Conn_01x08_Socket, J7 Conn_01x08_Socket, J8 Conn_01x19, J9 Conn_01x19

Commit message: cambios mayores
Parts:
- removed R10, R11, R7, R8, R9: 0, Resistor_THT:R_Axial_DIN0207_L6.3mm_D2.5mm_P10.16mm_Horizontal, symbol Device:R
- R1, R4, R6: footprint Resistor_SMD:R_1206_3216Metric_Pad1.30x1.75mm_HandSolder -> Resistor_THT:R_Axial_DIN0207_L6.3mm_D2.5mm_P10.16mm_Horizontal
Connections:
- net TCOL1 PWMB is gone; now on net TCOL2 PWMB: J6.7 (Pin_7)
- net GPIO02 5 TRIGGER 3: now also J3.2 (trigger)
- net GPIO2 6  TRIGGER 2: now also J1.2 (trigger)
- net TCOL0 PWMA: now also XA1.39 (tecCOL0)
- net servo: now reaches XA1.31 (tecCOL1)
- net servo: now also J5.1 (GNC)
- net TCOL2 PWMB: now reaches XA1.34 (tecCOL2)
- net TCOL2 PWMB: no longer J5.1 (GNC)
- net GPIO04  TRIGGER 1: now reaches XA1.73 (GPIO4)
- net GPIO04  TRIGGER 1: now also J2.2 (trigger)
- net GPIO05 12 TRIGGER 1: no longer names the net of XA1.64 (lcdRS)
Other:
- moved on the sheet: J5
