File: proyecto/car1/car1.kicad_pcb (KiCad board)
At the start: 2 copper layers, 137 x 85.9 mm, 29 parts, among them J1 HC-sr04, J10 vcc Edu ciaa, J11 Adafruit A, J12 Adafruit B, J2 HC-sr04, J3 HC-sr04, J4 usb c socket, J5 SERVO, J6 Conn_01x08_Socket, J7 Conn_01x08_Socket, J8 Conn_01x19, J9 Conn_01x19

Commit message: giga pad
Parts:
- moved C1 8.37 mm to (210.6, 58.0), turned to 0 degrees
- moved R7 1.02 mm to (195.3, 89.9)
Routing:
- net RS232_TX: track 54.4 -> 56.9 mm
- net GND: track 0.00 -> 2.29 mm
- net RS232_RX: track 55.3 -> 57.2 mm
- net TCOL0 PWMA: track 6.10 -> 7.33 mm
- net Net-(XA1A-tecCOL0): track 37.4 -> 36.4 mm
- net vcc: track 263.6 -> 262.9 mm

Commit message: fix pista
Routing:
- net TCOL0 PWMA: track 7.33 -> 5.53 mm
Changed lines of the file:
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@@
 	)
 	(segment
-		(start 197.866 101.346)
-		(end 196.596 101.346)
+		(start 195.326 100.076)
+		(end 197.866 100.076)
 		(width 0.7)
 		(layer "B.Cu")
@@
 	)
 	(segment
-		(start 198.897 97.511)
-		(end 198.897 100.315)
+		(start 197.866 100.076)
+		(end 198.897 99.045)
 		(width 0.7)
 		(layer "B.Cu")
@@
 	)
 	(segment
-		(start 198.897 100.315)
-		(end 197.866 101.346)
+		(start 198.897 99.045)
+		(end 198.897 97.511)
 		(width 0.7)
 		(layer "B.Cu")
-		(net 56)
-	)
-	(segment
-		(start 196.596 101.346)
-		(end 195.326 100.076)
-		(width 0.7)
-		(layer "B.Cu")
